Commit message: URDF for Body, New ROS Control

File: cnoid_tank_description/urdf/cnoid_tank.urdf.xacro (robot description, xacro)
@@ -19,11 +19,11 @@
     <child link ="Kinect_base"/>
   </joint>
-  <link name="Kinect"/>
+  <!-- <link name="Kinect"/>
   <joint name="Kinect" type="fixed">
     <origin rpy="${M_PI/2} ${M_PI} ${M_PI/2}"/>
     <parent link="Kinect_base"/>
     <child link="Kinect"/>
-  </joint>
-  <link name="VLP-16_base"/>
+  </joint> -->
+  <!-- <link name="VLP-16_base"/>
   <joint name="VLP-16_base" type="fixed">
     <origin xyz="0 0 0.225"/>
@@ -36,4 +36,4 @@
     <parent link="VLP-16_base"/>
     <child link="VLP-16"/>
-  </joint>
+  </joint> -->
 </robot>
